Commit message: no sliders

File: gp7_robot_description/urdf/gp7_robot.xacro (robot description, xacro)
@@ -2,7 +2,7 @@
   <link name="base_link">
     <inertial>
-      <origin xyz="0.00557004423686428 -1.25475368347918E-06 0.094757859890254" rpy="0 0 0" />
-      <mass value="5.21535720273169" />
-      <inertia ixx="0.0260255175058006" ixy="-2.60386335522236E-05" ixz="-0.000139873884034475" iyy="0.0252947855078615" iyz="4.77039729594201E-05" izz="0.0217201856002648" />
+      <origin xyz="0.00556892272669175 -6.27066159364017E-07 0.0947579647169003" rpy="0 0 0" />
+      <mass value="5.21544079925593" />
+      <inertia ixx="0.0260256781512797" ixy="-2.5924745904837E-05" ixz="-0.000139844593770951" iyy="0.0252950776511285" iyz="4.76784711767462E-05" izz="0.0217205299171908" />
     </inertial>
     <visual>
@@ -24,7 +24,7 @@
   <link name="link_1">
     <inertial>
-      <origin xyz="-0.0156633849726209 -0.000531476594167104 0.099849441027785" rpy="0 0 0" />
-      <mass value="2.94469808841832" />
-      <inertia ixx="0.0111825899978371" ixy="-3.08058902342631E-05" ixz="0.00217734244928747" iyy="0.0119457761701912" iyz="9.13688546392683E-05" izz="0.00886869098470957" />
+      <origin xyz="-0.0156640644370582 -0.000511078017811401 0.0998494406800811" rpy="0 0 0" />
+      <mass value="2.94469809358222" />
+      <inertia ixx="0.0111825110504346" ixy="-2.9811863375969E-05" ixz="0.00217745943510949" iyy="0.0119458549883966" iyz="8.85331651293519E-05" izz="0.00886869088704277" />
     </inertial>
     <visual>
@@ -49,11 +49,11 @@
     <child link="link_1" />
     <axis xyz="0 0 1" />
-    <limit lower="-3.1415" upper="3.1415" effort="50" velocity="1.0" />
+    <limit lower="0" upper="0" effort="0" velocity="0" />
   </joint>
   <link name="link_2">
     <inertial>
-      <origin xyz="0.0495045882226771 0.190602981532063 -0.00190315995896703" rpy="0 0 0" />
-      <mass value="6.24055262997388" />
-      <inertia ixx="0.125049731864705" ixy="-0.0109167450639977" ixz="-0.000630016577744454" iyy="0.0289782964319847" iyz="-2.0798262612872E-05" izz="0.110546834944449" />
+      <origin xyz="0.048951329816301 0.190746109963439 -0.00186791889973696" rpy="0 0 0" />
+      <mass value="6.2405514202476" />
+      <inertia ixx="0.12511389015047" ixy="-0.0106375502315048" ixz="-0.000612297490243357" iyy="0.0289157213719685" iyz="-4.65509655803263E-05" izz="0.110545180687341" />
     </inertial>
     <visual>
@@ -74,15 +74,15 @@
   </link>
   <joint name="joint_2" type="revolute">
-    <origin xyz="-0.039964 -0.0016995 0.1399" rpy="1.5708 0 0" />
+    <origin xyz="-0.0399638790462151 -0.00169952535722473 0.139900000000524" rpy="1.5707963267949 0 0" />
     <parent link="link_1" />
     <child link="link_2" />
-    <axis xyz="0.042488 0 0.9991" />
-    <limit lower="-3.1415" upper="3.1415" effort="50" velocity="1.0" />
+    <axis xyz="0.0412240631937652 0 0.999149926994841" />
+    <limit lower="0" upper="0" effort="0" velocity="0" />
   </joint>
   <link name="link_3">
     <inertial>
-      <origin xyz="0.0158049550440994 -0.0201368208412392 -0.00085391100684302" rpy="0 0 0" />
-      <mass value="2.84915098492796" />
-      <inertia ixx="0.00659554320497922" ixy="-0.000512367473814985" ixz="-3.08596154347593E-05" iyy="0.00857048171074949" iyz="3.716622638756E-05" izz="0.00779150072366676" />
+      <origin xyz="0.0160457922240239 -0.0190802860281885 -0.000816189919224628" rpy="0 0 0" />
+      <mass value="2.84915106810897" />
+      <inertia ixx="0.00658550295686827" ixy="-0.000492552305401648" ixz="-2.98557751860674E-05" iyy="0.0085806343455094" iyz="3.64668295071717E-05" izz="0.00779141136558319" />
     </inertial>
     <visual>
@@ -103,15 +103,15 @@
   </link>
   <joint name="joint_3" type="revolute">
-    <origin xyz="0.050376 0.44213 -0.0021423" rpy="0.041337 -0.0098821 1.8053" />
+    <origin xyz="0.0503759439359012 0.442134227086597 -0.002142314416107" rpy="0.041307778208651 -0.00969583648873429 1.80823908321343" />
     <parent link="link_2" />
     <child link="link_3" />
-    <axis xyz="0 0 -1" />
-    <limit lower="-3.1415" upper="3.1415" effort="50" velocity="1.0" />
+    <axis xyz="0 -0.0012296164180783 -0.999999243983334" />
+    <limit lower="0" upper="0" effort="0" velocity="0" />
   </joint>
   <link name="link_4">
     <inertial>
-      <origin xyz="-0.0401225094014942 -0.000183713948718249 0.245767638472074" rpy="0 0 0" />
-      <mass value="2.75537915804985" />
-      <inertia ixx="0.0101067865157806" ixy="-0.000122095516875289" ixz="5.92639216969416E-05" iyy="0.0107631491827932" iyz="-0.000313080392256919" izz="0.00308572026584051" />
+      <origin xyz="-0.00025976983308329 -0.000606527882467878 0.24675063483991" rpy="0 0 0" />
+      <mass value="2.75543476818323" />
+      <inertia ixx="0.010105688078101" ixy="-0.000119108463949627" ixz="5.78389419516153E-05" iyy="0.0107642324054807" iyz="-0.000313456642297312" izz="0.00308572821330252" />
     </inertial>
     <visual>
@@ -132,15 +132,15 @@
   </link>
   <joint name="joint_4" type="revolute">
-    <origin xyz="0.02 0 0" rpy="1.5708 0 2.9069" />
+    <origin xyz="0.0388801721925306 -0.00939797190787661 0.000454308759110602" rpy="1.57203865986274 0.000297435749113141 2.89685980999508" />
     <parent link="link_3" />
     <child link="link_4" />
     <axis xyz="0 0 1" />
-    <limit lower="-3.1415" upper="3.1415" effort="50" velocity="1.0" />
+    <limit lower="0" upper="0" effort="0" velocity="0" />
   </joint>
   <link name="link_5">
     <inertial>
-      <origin xyz="0.000253903122218069 0.0132104927332011 -0.00174847606756218" rpy="0 0 0" />
-      <mass value="0.24588630178433" />
-      <inertia ixx="0.000139534598690759" ixy="-2.11772918214912E-06" ixz="1.96190059856614E-07" iyy="0.000156835347164267" iyz="-1.29214828045847E-06" izz="0.000185616876010932" />
+      <origin xyz="-0.00310027636449783 0.0144406007119806 -0.00176602543910787" rpy="0 0 0" />
+      <mass value="0.245886306087054" />
+      <inertia ixx="0.000139576932998966" ixy="-2.28141914533607E-06" ixz="7.97120521965196E-10" iyy="0.000156791427083179" iyz="-1.2933551670261E-06" izz="0.000185618470305794" />
     </inertial>
     <visual>
@@ -161,15 +161,15 @@
   </link>
   <joint name="joint_5" type="revolute">
-    <origin xyz="-0.04 0 0.44" rpy="1.5708 -0.073037 0.17453" />
+    <origin xyz="0.00312213402888284 0.000136881955795811 0.439970310269017" rpy="1.57073179267725 -0.0658197300591794 0.174532730673124" />
     <parent link="link_4" />
     <child link="link_5" />
-    <axis xyz="0 0 1" />
-    <limit lower="-3.1415" upper="3.1415" effort="50" velocity="1.0" />
+    <axis xyz="-0.00447669926495448 0.000233060717240809 0.999989952372719" />
+    <limit lower="0" upper="0" effort="0" velocity="0" />
   </joint>
   <link name="link_6">
     <inertial>
-      <origin xyz="-1.44646797983761E-06 -7.38926903379178E-06 0.0851435220075776" rpy="0 0 0" />
-      <mass value="0.214725812821504" />
-      <inertia ixx="0.000223908058479713" ixy="-3.02140592461131E-05" ixz="3.99005585986096E-10" iyy="0.000132334918297617" iyz="2.03772760010368E-09" izz="0.000310945881078752" />
+      <origin xyz="-0.00407025472637845 3.23860923414909E-05 0.0863680824547134" rpy="0 0 0" />
+      <mass value="0.214725813088188" />
+      <inertia ixx="0.000223652589035899" ixy="-3.06090382841323E-05" ixz="-8.48310872937687E-07" iyy="0.000132598647310503" iyz="-2.46489126503789E-07" izz="0.00031093762188751" />
     </inertial>
     <visual>
@@ -190,15 +190,15 @@
   </link>
   <joint name="joint_6" type="revolute">
-    <origin xyz="0 0 0" rpy="-1.5708 0 0" />
+    <origin xyz="0 0 0" rpy="-1.5707963267949 0 0" />
     <parent link="link_5" />
     <child link="link_6" />
-    <axis xyz="0 0 -1" />
-    <limit lower="-3.1415" upper="3.1415" effort="50" velocity="1.0" />
+    <axis xyz="0.00982468830482129 -0.00029273971838837 -0.999951693734838" />
+    <limit lower="0" upper="0" effort="0" velocity="0" />
   </joint>
   <link name="link_7">
     <inertial>
-      <origin xyz="0 0.00410371116331321 -0.0210963244324723" rpy="0 0 0" />
-      <mass value="0.144760080963104" />
-      <inertia ixx="9.93365348547431E-05" ixy="-1.30443073877162E-19" ixz="6.26804380968182E-20" iyy="5.88881756954006E-05" iyz="1.81485780919137E-05" izz="0.000107613336062158" />
+      <origin xyz="-0.00442171967791183 0.00409624700892364 0.0178260368407184" rpy="0 0 0" />
+      <mass value="0.144760080963103" />
+      <inertia ixx="9.93343371743911E-05" ixy="-3.16311535090085E-07" ixz="2.07190731215265E-07" iyy="5.87984352111252E-05" iyz="1.80230086588129E-05" izz="0.000107705274226785" />
     </inertial>
     <visual>
@@ -219,15 +219,15 @@
   </link>
   <joint name="joint_7" type="prismatic">
-    <origin xyz="-0.011159 -0.037174 0.135" rpy="-1.5409 0 -0.29163" />
+    <origin xyz="-0.0111591245961624 -0.0371741770481596 0.135000000000577" rpy="-1.54088131317847 0 -0.29162636884829" />
     <parent link="link_6" />
     <child link="link_7" />
-    <axis xyz="0 -0.029911 -0.99955" />
-    <limit lower="0.0" upper="0.05" effort="20" velocity="0.1" />
+    <axis xyz="-0.00440449001661042 -0.0274111470578707 -0.999614540452802" />
+    <limit lower="0" upper="0" effort="0" velocity="0" />
   </joint>
   <link name="link_8">
     <inertial>
-      <origin xyz="0 0.00535780923501439 -0.0208131984585076" rpy="0 0 0" />
+      <origin xyz="0.00425198818078421 0.00284701261838405 0.020527996946165" rpy="0 0 0" />
       <mass value="0.144760080963103" />
-      <inertia ixx="9.93365348547428E-05" ixy="1.59453952320622E-19" ixz="-3.30342849429177E-20" iyy="5.689590477082E-05" iyz="1.51105268944253E-05" izz="0.000109605606986738" />
+      <inertia ixx="9.93316014788732E-05" ixy="4.6896953643637E-07" ixz="-1.05074443727185E-07" iyy="5.69782736000298E-05" iyz="1.52440684406542E-05" izz="0.000109528171533398" />
     </inertial>
     <visual>
@@ -248,9 +248,9 @@
   </link>
   <joint name="joint_8" type="prismatic">
-    <origin xyz="0.011159 0.037174 0.135" rpy="-1.6007 0 2.85" />
+    <origin xyz="0.0111591245878672 0.0371741770439874 0.134999999999424" rpy="-1.60071134041132 0 2.8499662847415" />
     <parent link="link_6" />
     <child link="link_8" />
-    <axis xyz="0 -0.029911 0.99955" />
-    <limit lower="0.0" upper="0.05" effort="20" velocity="0.1" />
+    <axis xyz="0.00440449001661078 -0.0274111470578707 0.999614540452801" />
+    <limit lower="0" upper="0" effort="0" velocity="0" />
   </joint>
 </robot>
